File: PCB/KiCad/IsoDiffProbe.kicad_pcb (KiCad board)
At the start: 2 copper layers, 77.2 x 49.1 mm, 79 parts, among them J1 USB C 6-Pin, J2 SMA Conn, P1 Header 10X2, U1 AMC3, U2 TLC272ID

Commit message: Clean Altium file. REv A1 mods
Parts:
- D1, D2: footprint Genesis_PCB_Footprints.PcbLib:LED-0603 -> E GF.PcbLib:LED-0603
- P1: footprint EDMI Altium Connectors.PcbLib:IDC20 -> E Connectors.PcbLib:IDC20
- R15, R23, R26, R27, R31, R32: footprint EDMI Altium General Footprints.PcbLib:MMB0207 -> E General.PcbLib:MMB0207
- TP1, TP10, TP11, TP12, TP13, TP14, TP15, TP16, TP17, TP18, TP19, TP2, TP20, TP3, TP4, TP5, TP6, TP7, TP8, TP9: footprint EDMI Altium General Footprints.PcbLib:TP -> E General.PcbLib:TP
- U1: footprint Genesis_PCB_Footprints.PcbLib:DW0016B -> E GF.PcbLib:DW0016B
- U2: footprint EDMI Altium General Footprints.PcbLib:SO-8 -> E General.PcbLib:SO-8
Changed lines of the file:
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@@
 		)
 	)
+	(property "ENGINEER" "Michael")
+	(property "SHEETTOTAL" "1")
 	(net 0 "")
 	(net 1 "ISOLDO")
@@
 		)
 		(property "Value" "10pF"
-			(at -0.3937 3.0353 270)
+			(at -0.3937 3.0353 -90)
 			(unlocked yes)
 			(layer "F.SilkS")
@@
 		)
 		(property "Value" "1nF"
-			(at -2.9337 -0.4953 270)
+			(at -2.9337 -0.4953 -90)
 			(unlocked yes)
 			(layer "F.SilkS")
@@
 		)
 		(property "Value" "11k"
-			(at -2.9337 -0.4953 270)
+			(at -2.9337 -0.4953 -90)
 			(unlocked yes)
 			(layer "F.SilkS")
@@
 		)
 		(property "Value" "4k7"
-			(at -3.1877 -0.9017 270)
+			(at -3.1877 -0.9017 -90)
 			(unlocked yes)
 			(layer "F.SilkS")
@@
 		)
 		(property "Value" "100nF"
-			(at -2.9337 -0.4953 270)
+			(at -2.9337 -0.4953 -90)
 			(unlocked yes)
 			(layer "F.SilkS")
@@
 		)
 	)
-	(footprint "EDMI Altium General Footprints.PcbLib:MMB0207"
+	(footprint "E General.PcbLib:MMB0207"
 		(layer "F.Cu")
 		(at 125.7261 118.7411)
@@
 		)
 		(property "Value" "470k"
-			(at -3.8481 -1.5367 270)
+			(at -3.8481 -1.5367 -90)
 			(unlocked yes)
 			(layer "F.SilkS")
@@
 		)
 	)
-	(footprint "EDMI Altium General Footprints.PcbLib:TP"
+	(footprint "E General.PcbLib:TP"
 		(layer "F.Cu")
 		(at 159.8811 106.3461 90)
@@
 		)
 	)
-	(footprint "EDMI Altium General Footprints.PcbLib:TP"
+	(footprint "E General.PcbLib:TP"
 		(layer "F.Cu")
 		(at 112.1461 90.7811)
@@
 		)
 	)
-	(footprint "EDMI Altium General Footprints.PcbLib:MMB0207"
+	(footprint "E General.PcbLib:MMB0207"
 		(layer "F.Cu")
 		(at 117.5261 126.3411)
@@
 		)
 		(property "Value" "470k"
-			(at -3.8481 -1.5367 270)
+			(at -3.8481 -1.5367 -90)
 			(unlocked yes)
 			(layer "F.SilkS")
@@
 		)
 	)
-	(footprint "EDMI Altium General Footprints.PcbLib:TP"
+	(footprint "E General.PcbLib:TP"
 		(layer "F.Cu")
 		(at 112.1461 98.4011)
@@
 		)
 		(property "Value" "10k"
-			(at -2.93369 -0.4953 270)
+			(at -2.93369 -0.4953 -90)
 			(unlocked yes)
 			(layer "F.SilkS")
@@
 		)
 		(property "Value" "100nF"
-			(at -0.3937 3.0353 270)
+			(at -0.3937 3.0353 -90)
 			(unlocked yes)
 			(layer "F.SilkS")
@@
 		)
 	)
-	(footprint "EDMI Altium General Footprints.PcbLib:MMB0207"
+	(footprint "E General.PcbLib:MMB0207"
 		(layer "F.Cu")
 		(at 117.5261 106.0411)
@@
 		)
 		(property "Value" "470k"
-			(at -3.8481 -1.5367 270)
+			(at -3.8481 -1.5367 -90)
 			(unlocked yes)
 			(layer "F.SilkS")
@@
 		)
 	)
-	(footprint "EDMI Altium General Footprints.PcbLib:TP"
+	(footprint "E General.PcbLib:TP"
 		(layer "F.Cu")
 		(at 173.5061 95.1411)
@@
 		)
 	)
-	(footprint "EDMI Altium General Footprints.PcbLib:TP"
+	(footprint "E General.PcbLib:TP"
 		(layer "F.Cu")
 		(at 159.8811 101.2661 90)
@@
 		)
 	)
-	(footprint "EDMI Altium General Footprints.PcbLib:TP"
+	(footprint "E General.PcbLib:TP"
 		(layer "F.Cu")
 		(at 173.5061 110.3811 90)
@@
 		)
 	)
-	(footprint "Genesis_PCB_Footprints.PcbLib:DW0016B"
+	(footprint "E GF.PcbLib:DW0016B"
 		(layer "F.Cu")
 		(at 151.3481 98.5471)
@@
 		)
 		(property "Value" "4k7"
-			(at -3.1877 -0.9017 270)
+			(at -3.1877 -0.9017 -90)
 			(unlocked yes)
 			(layer "F.SilkS")
@@
 		)
 	)
-	(footprint "EDMI Altium General Footprints.PcbLib:MMB0207"
+	(footprint "E General.PcbLib:MMB0207"
 		(layer "F.Cu")
 		(at 125.7261 126.3411)
@@
 		)
 		(property "Value" "470k"
-			(at -3.8481 -1.5367 270)
+			(at -3.8481 -1.5367 -90)
 			(unlocked yes)
 			(layer "F.SilkS")
@@
 		)
 	)
-	(footprint "EDMI Altium General Footprints.PcbLib:MMB0207"
+	(footprint "E General.PcbLib:MMB0207"
 		(layer "F.Cu")
 		(at 117.5261 118.7411)
@@
 		)
 		(property "Value" "470k"
-			(at -3.8481 -1.5367 270)
+			(at -3.8481 -1.5367 -90)
 			(unlocked yes)
 			(layer "F.SilkS")
@@
 		)
 	)
-	(footprint "EDMI Altium General Footprints.PcbLib:TP"
+	(footprint "E General.PcbLib:TP"
 		(layer "F.Cu")
 		(at 138.5621 93.5751 -90)
@@
 		(fp_arc
 			(start 7.492 -3.69999)
-			(mid 7.85121 -3.5512)
+			(mid 7.851207 -3.5512)
 			(end 8 -3.19199)
 			(stroke
@@
 		(fp_arc
 			(start 1.508 -3.69999)
-			(mid 1.864371 -3.554017)
+			(mid 1.864368 -3.554016)
 			(end 2.015937 -3.199988)
 			(stroke
@@
 		(fp_arc
 			(start 6.984063 -3.199988)
-			(mid 7.135629 -3.554017)
+			(mid 7.135625 -3.554023)
 			(end 7.492 -3.69999)
 			(stroke
@@
 		)
 	)
-	(footprint "EDMI Altium General Footprints.PcbLib:TP"
+	(footprint "E General.PcbLib:TP"
 		(layer "F.Cu")
 		(at 112.1461 93.3211)
@@
 		)
 	)
-	(footprint "EDMI Altium General Footprints.PcbLib:TP"
+	(footprint "E General.PcbLib:TP"
 		(layer "F.Cu")
 		(at 173.5061 100.2211)
@@
 		)
 	)
-	(footprint "EDMI Altium General Footprints.PcbLib:TP"
+	(footprint "E General.PcbLib:TP"
 		(layer "F.Cu")
 		(at 112.1461 126.3411 90)
@@
 		)
 	)
-	(footprint "EDMI Altium General Footprints.PcbLib:MMB0207"
+	(footprint "E General.PcbLib:MMB0207"
 		(layer "F.Cu")
 		(at 117.5261 111.1411)
@@
 		)
 		(property "Value" "470k"
-			(at -3.8481 -1.5367 270)
+			(at -3.8481 -1.5367 -90)
 			(unlocked yes)
 			(layer "F.SilkS")
@@
 		)
 	)
-	(footprint "EDMI Altium Connectors.PcbLib:IDC20"
+	(footprint "E Connectors.PcbLib:IDC20"
 		(layer "F.Cu")
 		(at 130.9421 85.9551 -90)
@@
 		)
 	)
-	(footprint "EDMI Altium General Footprints.PcbLib:TP"
+	(footprint "E General.PcbLib:TP"
 		(layer "F.Cu")
 		(at 112.1461 100.9411)
@@
 		)
 	)
-	(footprint "EDMI Altium General Footprints.PcbLib:TP"
+	(footprint "E General.PcbLib:TP"
 		(layer "F.Cu")
 		(at 112.1461 118.7211 90)
@@
 		)
 	)
-	(footprint "EDMI Altium General Footprints.PcbLib:TP"
+	(footprint "E General.PcbLib:TP"
 		(layer "F.Cu")
 		(at 112.1461 85.7011)
@@
 		)
 		(property "Value" "10k"
-			(at -2.9337 -0.4953 270)
+			(at -2.9337 -0.4953 -90)
 			(unlocked yes)
 			(layer "F.SilkS")
@@
 		)
 	)
-	(footprint "EDMI Altium General Footprints.PcbLib:TP"
+	(footprint "E General.PcbLib:TP"
 		(layer "F.Cu")
 		(at 138.5621 91.0351 -90)
@@
 		)
 	)
-	(footprint "EDMI Altium General Footprints.PcbLib:SO-8"
+	(footprint "E General.PcbLib:SO-8"
 		(layer "F.Cu")
 		(at 163.23611 113.6291 90)
@@
 		)
 	)
-	(footprint "Genesis_PCB_Footprints.PcbLib:LED-0603"
+	(footprint "E GF.PcbLib:LED-0603"
 		(layer "F.Cu")
 		(at 164.0511 95.3161 180)
@@
 		)
 	)
-	(footprint "Genesis_PCB_Footprints.PcbLib:LED-0603"
+	(footprint "E GF.PcbLib:LED-0603"
 		(layer "F.Cu")
 		(at 164.05109 97.6661 180)
@@
 		)
 		(property "Value" "100nF"
-			(at -2.9337 -0.4953 270)
+			(at -2.9337 -0.4953 -90)
 			(unlocked yes)
 			(layer "F.SilkS")
@@
 		)
 		(property "Value" "PBY201209T-601Y-N"
-			(at -0.6985 3.2639 270)
+			(at -0.6985 3.2639 -90)
 			(unlocked yes)
 			(layer "F.SilkS")
@@
 		)
 		(property "Value" "5k1"
-			(at -0.3937 3.0353 270)
+			(at -0.3937 3.0353 -90)
 			(unlocked yes)
 			(layer "F.SilkS")
@@
 		)
 	)
-	(footprint "EDMI Altium General Footprints.PcbLib:TP"
+	(footprint "E General.PcbLib:TP"
 		(layer "F.Cu")
 		(at 112.1461 83.1611)
@@
 		)
 		(property "Value" "NF"
-			(at -0.3937 3.0353 270)
+			(at -0.3937 3.0353 -90)
 			(unlocked yes)
 			(layer "F.SilkS")
@@
 		)
 		(property "Value" "10uF / 25V"
-			(at -0.4953 3.2639 270)
+			(at -0.4953 3.2639 -90)
 			(unlocked yes)
 			(layer "F.SilkS")
@@
 		)
 	)
-	(footprint "EDMI Altium General Footprints.PcbLib:TP"
+	(footprint "E General.PcbLib:TP"
 		(layer "F.Cu")
 		(at 159.8811 103.8061 90)
@@
 		)
 	)
-	(footprint "EDMI Altium General Footprints.PcbLib:TP"
+	(footprint "E General.PcbLib:TP"
 		(layer "F.Cu")
 		(at 173.5061 115.4611 90)
@@
 		)
 	)
-	(footprint "EDMI Altium General Footprints.PcbLib:TP"
+	(footprint "E General.PcbLib:TP"
 		(layer "F.Cu")
 		(at 138.5621 96.1151 -90)
@@
 		)
 		(property "Value" "51k"
-			(at -3.1877 -0.9017 270)
+			(at -3.1877 -0.9017 -90)
 			(unlocked yes)
 			(layer "F.SilkS")
@@
 		)
 		(property "Value" "NF"
-			(at -0.3937 3.0353 270)
+			(at -0.3937 3.0353 -90)
 			(unlocked yes)
 			(layer "F.SilkS")
@@
 		)
 		(property "Value" "51k"
-			(at -3.1877 -0.9017 270)
+			(at -3.1877 -0.9017 -90)
 			(unlocked yes)
 			(layer "F.SilkS")
@@
 		)
 		(property "Value" "NF"
-			(at -0.3937 3.0353 270)
+			(at -0.3937 3.0353 -90)
 			(unlocked yes)
 			(layer "F.SilkS")
@@
 		)
 	)
-	(footprint "EDMI Altium General Footprints.PcbLib:TP"
+	(footprint "E General.PcbLib:TP"
 		(layer "F.Cu")
 		(at 112.1461 111.1011 90)
@@
 		)
 	)
-	(footprint "EDMI Altium General Footprints.PcbLib:TP"
+	(footprint "E General.PcbLib:TP"
 		(layer "F.Cu")
 		(at 112.1461 106.0211)
@@
 		)
 		(property "Value" "100nF"
-			(at -0.3937 3.0353 270)
+			(at -0.3937 3.0353 -90)
 			(unlocked yes)
 			(layer "F.SilkS")
@@
 	)
 	(gr_rect
-		(start 180.3011 116.4661)
-		(end 180.9261 114.2161)
+		(start 180.3011 114.2161)
+		(end 180.9261 116.4661)
 		(stroke
 			(width 0)
@@
 	)
 	(gr_rect
-		(start 180.3761 107.8161)
-		(end 180.9761 105.5661)
+		(start 180.3761 105.5661)
+		(end 180.9761 107.8161)
 		(stroke
 			(width 0)
@@
 	)
 	(gr_rect
-		(start 187.05111 114.8161)
-		(end 180.65111 114.2161)
+		(start 180.65111 114.2161)
+		(end 187.05111 114.8161)
 		(stroke
 			(width 0)
@@
 	)
 	(gr_rect
-		(start 187.05111 114.8161)
-		(end 180.65111 114.2161)
+		(start 180.65111 114.2161)
+		(end 187.05111 114.8161)
 		(stroke
 			(width 0)
