File: KiCad rev B/IsoDiffProbe_B.kicad_sch (KiCad schematic)
At the start: 82 parts, among them J1 USB C 6-Pin, J2 SMA Conn, P1 Header 10X2, U1 AMC33xx, U2 OPA2376

Commit message: Value changes to improve rev A1->A2 and updated rev B design.
Parts:
- added C21: 33pF, NixieClock_RevA.PcbLib:0603, symbol IsoDiffProbe-altium-import:root_0_mirrored_CAP-STD-SM
- added D3: MRA4007T3G, Diode_SMD:D_SMA, symbol Diode:MRA4007T3G
- added R35, R36: 1k, NixieClock_RevA.PcbLib:1206, symbol IsoDiffProbe-altium-import:root_0_RES-SM
- C1: value NF -> 100nF
- C11: value 10pF -> 33pF
- C12, C15: value 100pF -> 33pF
- C19: value 82pF -> 100pF
- C20: value 1nF Y1 -> 33pF
- P1: Function (none) -> Input Selection
- R11, R13: value 220R -> 22R
Connections:
- net GND: now also D3.2 (A); no longer C20.2
- net HGND: now also C21.2
- net VIN: now also D3.1 (K)
- net at C11.1, R11.1, U1.6 (INP): now also C20.2, R34.1
- net at P1.10, P1.14, P1.18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: no longer R34.1
- net at C11.2, R13.1, U1.7 (INN): now also R33.1, C21.1
- net at C1.1, R1.2, TP1.1 (0): now also R35.1; no longer P1.1
- net at C1.2, R1.1, TP2.1 (0): now also R36.1; no longer P1.3
- net at P1.12, P1.16, P1.20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: no longer R33.1
- new net: P1.1, R35.2
- new net: P1.3, R36.2
Other:
- note added: "*"
- note added: "* = Not currently on RevB PCB"
- note added: "Filter & bias values depend on U1: U1=AMC3300 (Voltage probe): R34,R33=1M and C11,C20,C21=33pF U1=AMC3301 (Current probe): R34,R33=100k and C11,C20,C21=3.3nF All except C11 are new in RevB"
- note added: "For U1=AMC3302 multi-shunt input, place shunt at ends of input resistor=0R, eg:"
- note added: "fc ≈ 200-300kHz"
- note added: "https://github.com/michael0093/Isolated-Diff-Probe"
- note removed: "fc = 1.49MHz"
- note removed: "fc = 1.60MHz"
- note removed: "fc = 1.61MHz"
- note removed: "fc = 916kHz"
- moved on the sheet: R11, R13, R33, R34, TP6, TP7
